Commit message: simulator: Change basic body mesh to gokart mesh

File: simulator/urdf/ackermann.urdf (robot description, URDF)
Before this commit: robot gokart, 3 links, 2 joints
Links:
- link base_link: geometry collision box size=${base_length} ${base_width} ${base_height}; visual mesh filename=file://$(find simulator)/meshes/gokart/BodyV1.stl

Commit message: simulator: Update simulation (add sensors to model)

File: simulator/urdf/ackermann.urdf (robot description, URDF)
Before this commit: robot gokart, 3 links, 2 joints
Links:
- added link lidar_link, mass 0.125; collision cylinder length=0.75 radius=0.0508; visual cylinder length=0.75 radius=0.0508
Joints:
- added joint lidar_joint: type fixed, parent base_link, child lidar_link, origin xyz=0.215 0.0 0.30 rpy=0 0 0
