Commit message: simulation: Refactor simulator_gazebo_plugin and simulator

File: simulator/urdf/gokart.urdf (robot description, URDF)
Before this commit: robot gokart, 6 links, 5 joints
Links:
- removed link front_caster
- link base_link: geometry collision box size=${base_length} ${base_width} ${base_height}; visual mesh filename=file://$(find simulator)/meshes/gokart/BodyV1.stl
Joints:
- removed joint caster_joint

Commit message: simulator: Change base_link position, delete root_link in the gokart URDF

File: simulator/urdf/gokart.urdf (robot description, URDF)
Before this commit: robot gokart, 5 links, 4 joints
Links:
- removed link base_footprint
- removed link root_link
- added link body_frame_link; collision box size=${base_length} ${base_width-steering_hinge_offset-0.15} ${b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; visual mesh filename=file://$(find simulator)/meshes/gokart/BodyV1.stl
- link base_link: geometry 
Joints:
- removed joint base_joint
- removed joint root_joint
- added joint body_frame_joint: type fixed, parent base_link, child body_frame_link, origin xyz=0.525 0.0 0.0 rpy=0 0 0
- joint imu_joint: origin xyz=0 0 0.01 -> xyz=0.5 0 0.01
- joint lidar_joint: origin xyz=0.215 0.0 0.30 rpy=0 0 0 -> xyz=0.715 0.0 0.30 rpy=0 0 0

Commit message: simulator: Add camera sensor to gokart simulation

File: simulator/urdf/gokart.urdf (robot description, URDF)
Before this commit: robot gokart, 4 links, 3 joints
Links:
- added link camera_link; visual box size=0.03 0.2 0.03
Joints:
- added joint camera_joint: type fixed, parent base_link, child camera_link, origin xyz=0.755 0.0 0.30 rpy=0 0 0
